Commit message: partial rewrite

File: xacro/gazebo_control.xacro (robot description, xacro)
@@ -3,7 +3,7 @@
     <!-- PLUGINS -->
     <gazebo>
-        <plugin name="${robot_name}_joint_state" filename="libgazebo_ros_joint_state_publisher.so">
+        <plugin name="joint_state" filename="libgazebo_ros_joint_state_publisher.so">
             <ros>
-                <namespace>/${robot_name}</namespace>
+                <namespace>${robot_name}</namespace>
                 <!-- <remapping>~/out:=joint_states</remapping> -->
             </ros>
@@ -19,7 +19,7 @@
     <!-- Differential drive -->
     <gazebo>
-        <plugin filename="libgazebo_ros_diff_drive.so" name="${robot_name}_differential_drive_controller">
+        <plugin filename="libgazebo_ros_diff_drive.so" name="differential_drive_controller">
         <ros>
-            <namespace>/${robot_name}</namespace>
+            <namespace>${robot_name}</namespace>
             <!--
                 <argument> -ros-args -remap /cmd_vel:=/${robot_name}/cmd_vel /odom:=/${robot_name}/odom</argument>

File: xacro/properties.xacro (robot description, xacro)
@@ -26,11 +26,3 @@
     <xacro:property name="lidar_zoff" value="-0.0273"/>
     <!-- <xacro:property name="lidar_zoff" value="-0.06"/> -->
-    <!-- Camera -->
-    <xacro:property name="camera_xoff" value="0.4972"/>
-    <xacro:property name="camera_yoff" value="0.0"/>
-    <xacro:property name="camera_zoff" value="0.0298"/>
-    <xacro:property name="camera_depth_width" value="640"/>
-    <xacro:property name="camera_depth_height" value="480"/>
-    <xacro:property name="camera_color_width" value="640"/>
-    <xacro:property name="camera_color_height" value="480"/>
 </robot>

File: xacro/vikings_bot.xacro (robot description, xacro)
@@ -14,5 +14,4 @@
     <xacro:include filename="$(find vikings_bot_description)/xacro/wheels.xacro"/>
     <xacro:include filename="$(find vikings_bot_description)/xacro/castor_wheels.xacro"/>
-    <xacro:include filename="$(find realsense2_description)/urdf/_d415.urdf.xacro"/>
     <!-- Include Gazebo related files -->
     <!-- ROBOT -->
@@ -121,19 +120,4 @@
         <origin xyz="${lidar_xoff} ${lidar_yoff} ${lidar_zoff}" rpy="0 0 0"/>
     </joint>
-    <!-- Camera -->
-    <!-- realsense2_description package manages camera's description (geometry etc.) -->
-    <!--TODO: add use sim time parameter to use_nominal_extrinsics (should only be true in sim)-->
-    <xacro:sensor_d415 parent="chassis_link" use_nominal_extrinsics="${use_sim}">
-        <origin xyz="${camera_xoff} ${camera_yoff} ${camera_zoff}" rpy="0 0 0"/>
-    </xacro:sensor_d415>
-    <gazebo reference="camera_link">
-        <material>Gazebo/Grey</material>
-        <!-- friction -->
-        <mu1>100</mu1>
-        <mu2>100</mu2>
-        <!-- stiffness -->
-        <kp>100000000000000000</kp>
-        <kd>100000000000000000</kd>
-    </gazebo>
     <!-- If use "use_sim "-->
     <xacro:if value="${use_sim}">
@@ -173,5 +157,5 @@
                 </noise>
             </ray>
-            <plugin name="${robot_name}_lidar_scan" filename="libgazebo_ros_ray_sensor.so">
+            <plugin name="lidar_scan" filename="libgazebo_ros_ray_sensor.so">
                 <ros>
                     <namespace>${robot_name}</namespace>
@@ -183,128 +167,3 @@
         </sensor>
     </gazebo>
-   <!-- Camera sensor -->
-   <!--
-    uses pal robotics realsense_gazebo_plugin
-    https://github.com/pal-robotics/realsense_gazebo_plugin/tree/foxy-devel
-   -->
-   <gazebo reference="camera_link">
-    <sensor name="cameradepth" type="depth">
-        <camera name="camera">
-          <horizontal_fov>1.57</horizontal_fov>
-          <image>
-            <width>${camera_depth_width}</width>
-            <height>${camera_depth_height}</height>
-          </image>
-          <clip>
-            <near>0.1</near>
-            <far>100</far>
-          </clip>
-          <noise>
-            <type>gaussian</type>
-            <mean>0.0</mean>
-            <stddev>0.100</stddev>
-          </noise>
-        </camera>
-        <always_on>1</always_on>
-        <update_rate>30</update_rate>
-        <visualize>0</visualize>
-      </sensor>
-      <sensor name="cameracolor" type="camera">
-        <camera name="camera">
-          <horizontal_fov>1.57</horizontal_fov>
-          <image>
-            <width>${camera_color_width}</width>
-            <height>${camera_color_height}</height>
-            <format>RGB_INT8</format>
-          </image>
-          <clip>
-            <near>0.1</near>
-            <far>100</far>
-          </clip>
-          <noise>
-            <type>gaussian</type>
-            <mean>0.0</mean>
-            <stddev>0.007</stddev>
-          </noise>
-        </camera>
-        <always_on>1</always_on>
-        <update_rate>30</update_rate>
-        <visualize>1</visualize>
-      </sensor>
-      <sensor name="cameraired1" type="camera">
-        <camera name="camera">
-          <horizontal_fov>1.57</horizontal_fov>
-          <image>
-            <width>${camera_depth_width}</width>
-            <height>${camera_depth_height}</height>
-            <format>L_INT8</format>
-          </image>
-          <clip>
-            <near>0.1</near>
-            <far>100</far>
-          </clip>
-          <noise>
-            <type>gaussian</type>
-            <mean>0.0</mean>
-            <stddev>0.05</stddev>
-          </noise>
-        </camera>
-        <always_on>1</always_on>
-        <update_rate>1</update_rate>
-        <visualize>0</visualize>
-      </sensor>
-      <sensor name="cameraired2" type="camera">
-        <camera name="camera">
-          <horizontal_fov>1.57</horizontal_fov>
-          <image>
-            <width>${camera_depth_width}</width>
-            <height>${camera_depth_height}</height>
-            <format>L_INT8</format>
-          </image>
-          <clip>
-            <near>0.1</near>
-            <far>100</far>
-          </clip>
-          <noise>
-            <type>gaussian</type>
-            <mean>0.0</mean>
-            <stddev>0.05</stddev>
-          </noise>
-        </camera>
-        <always_on>1</always_on>
-        <update_rate>1</update_rate>
-        <visualize>0</visualize>
-      </sensor>
-   </gazebo>
-   <gazebo>
-    <plugin name="${robot_name}_camera" filename="librealsense_gazebo_plugin.so">
-        <prefix>camera</prefix>
-        <!--
-            actual FPS (and publishing rate, Hz) is 6 (at 1280x720) for realsense depth module.
-            Plugin caps depth FPS at 6. To increase FPS, change resolution in properties.xacro
-        -->
-        <depthUpdateRate>30.0</depthUpdateRate>
-        <colorUpdateRate>30.0</colorUpdateRate>
-        <infraredUpdateRate>1.0</infraredUpdateRate>
-        <!-- realsense uses aligned depth to color topic. For sim assume that default depth topic is aligned with color frame-->
-        <depthTopicName>${robot_name}/camera/aligned_depth_to_color/image_raw</depthTopicName>
-      	<depthCameraInfoTopicName>${robot_name}/camera/depth/camera_info</depthCameraInfoTopicName>
-      	<colorTopicName>${robot_name}/camera/color/image_raw</colorTopicName>
-      	<colorCameraInfoTopicName>${robot_name}/camera/color/camera_info</colorCameraInfoTopicName>
-        <!--real realsense camera does not publish infared image topics, but removing these params breaks the plugin-->
-      	<infrared1TopicName>${robot_name}/camera/infra1/image_raw</infrared1TopicName>
-      	<infrared1CameraInfoTopicName>${robot_name}/camera/infra1/camera_info</infrared1CameraInfoTopicName>
-      	<infrared2TopicName>${robot_name}/infra2/image_raw</infrared2TopicName>
-      	<infrared2CameraInfoTopicName>${robot_name}/camera/infra2/camera_info</infrared2CameraInfoTopicName>
-        <colorOpticalframeName>${robot_name}/camera_color_optical_frame</colorOpticalframeName>
-        <depthOpticalframeName>${robot_name}/camera_depth_optical_frame</depthOpticalframeName>
-        <infrared1OpticalframeName>${robot_name}/camera_left_ir_optical_frame</infrared1OpticalframeName>
-        <infrared2OpticalframeName>${robot_name}/camera_right_ir_optical_frame</infrared2OpticalframeName>
-        <rangeMinDepth>0.3</rangeMinDepth>
-        <rangeMaxDepth>3.0</rangeMaxDepth>
-        <pointCloud>true</pointCloud>
-        <pointCloudTopicName>${robot_name}/camera/depth/color/points</pointCloudTopicName>
-        <pointCloudCutoff>0.3</pointCloudCutoff>
-    </plugin>
-   </gazebo>
 </robot>
